File: fan-lpc11u24/fanbot.sch (KiCad schematic (older format))
At the start: 59 parts, among them K1 CONN_3, K2 CONN_3, P1 CONN_4, P2 CONN_6, P3 CONN_6, P4 CONN_5, P5 CONN_4, P6 CONN_6, P7 CONN_4, P8 CONN_4, SW1 Tactile push, U1 NX1117CE33Z, U2 LPC11U24FBD48/301, U3 GP1UX310QS, X1 12MHz

Commit message: Added test pins for unused uC pins, fixed USB pinning
Parts:
- added TP1, TP10, TP11, TP12, TP2, TP3, TP4, TP5, TP6, TP7, TP8, TP9: CONN_1, symbol CONN_1
- R3, R8: value 68R -> 33R; Farnell 9233865 -> 9233822; MFG PHYCOMP-RC0805JR-0768RL -> PHYCOMP-RC0805JR-0733RL
Connections:
- net labels added: TP1, TP10, TP11, TP12, TP2, TP3, TP4, TP5, TP6, TP7, TP8, TP9
- wire segments 112 -> 136
Other:
- note added: "Face LEDs"
- note added: "ISP Enable (USB MSD mode)"
- note added: "RC Servo outputs"
- note added: "Test pins (unused uC)"
- note removed: "1"
- note removed: "ISP Enable"
- moved on the sheet: D1, D2, D4, D5, D6, D7, D8, K2, R1, R11, R12, R13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

Commit message: Fixed pinning of servo connectors
Parts:
- renumbered TP1 to T1, TP10 to T10, TP11 to T11, TP12 to T12, TP2 to T2, TP3 to T3, TP4 to T4, TP5 to T5, TP6 to T6, TP7 to T7, TP8 to T8, TP9 to T9
Connections:
- wire segments 136 -> 134
Other:
- moved on the sheet: R3, R8
