File: fan-lpc11u24/fanbot.sch (KiCad schematic (older format))
At the start: 71 parts, among them K1 CONN_3, K2 CONN_3, P1 CONN_4, P2 CONN_6, P3 CONN_6, P4 CONN_5, P5 CONN_4, P6 CONN_6, P7 CONN_4, P8 CONN_4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

Commit message: Added pictures
Parts:
- removed T8: CONN_1, symbol CONN_1
- added Q1: BSS84, symbol MOSFET_P
- R18: value 4.7k -> 43k; Farnell 2074469 -> 2073781; MFG MULTICOMP-MCSR08X4701FTL -> MULTICOMP-MCMR08X4702FTL (1%)
Connections:
- net labels added: USB_CON
- net labels removed: TP8
- wire segments 134 -> 135
Other:
- note added: "45 Ohm impedance / 90 Ohm differential routing"
- note added: "Avoid stubs / ground plane crossovers"
- note added: "No traces < 5width to USB lines"
- moved on the sheet: C13, C14, P5, R17, R19

Commit message: changed schematic for USB, not routed yet
Parts:
- JP1: value USB-B -> USB-B (micro)
Connections:
- wire segments 135 -> 141
Other:
- note added: "Center"
- note added: "DNA"
- note added: "Expansion connectors (optional) 2.54mm\n"
- note added: "IR link (optional). 38kHz, through hole components (2.54mm)"
- note added: "Left eye"
- note added: "Left mouth"
- note added: "Right eye\n"
- note added: "Right mouth\n"
- note added: "SWD debug connection (2.54mm)\n"
- note removed: "Expansion connectors\n"
- note removed: "IR link (optional)"
- note removed: "SWD debug connection\n"
- moved on the sheet: C1, C2, C6, D1, D2, D4, D5, D6, D7, D8, K1, K2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
