File: hub/fanbot-hub.sch (KiCad schematic (older format))
At the start: 121 parts, among them J1 USBA-D, J10 USBA-D, J11 USBA-D, J12 USBA-D, J13 RJ45IN, J14 RJ45OUT, J15 USB_1, J2 USBA-D, J3 USBA-D, J4 USBA-D, J5 USBA-D, J6 USBA-D, J7 USBA-D, J8 USBA-D, J9 USBA-D, P1 POWER, P2 POWER, Q1 BSS84, SW1 SPST, SW2 SPST, SW3 DIPS_04, U1 NX1117CE33Z, U2 ADM2484, U3 NX1117CE50Z, U4 LPC11U35FBD64/401

Commit message: Created output files
Parts:
- removed J15: USB_1, symbol USB_1
- added C19, C20: 10000uF, symbol CAPAPOL
- added C21, C22: 18pF, symbol CSMALL
- added J15: USB, symbol USB
- added X1: 12MHz, symbol CRYSTAL
- C18: renamed from 100nF1; value C -> 100nF
Connections:
- wire segments 236 -> 241
Other:
- moved on the sheet: C10, C11, C12, C13, C14, C15, C3, C4, C5, C9, Q1, R16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

Commit message: Added crystal and capacitors
Parts:
- added D8: DIODE, symbol DIODE
- added JP1: JUMPER, symbol JUMPER
Other:
- moved on the sheet: C15, R19

Commit message: Added pictures
Parts:
- removed F10, F12, F14, F16, F18, F2, F20, F22, F24, F4, F6, F8: 1.25A, 1812, symbol FUSE
- added FB?: FILTER, symbol FILTER
- added FB? (x2): 0.1R / 1A, symbol FILTER
- added P?: POWER, symbol CONN_2
Connections:
- net labels added: V1, V10, V11, V12, V2, V3, V4, V5, V6, V7, V8, V9
- wire segments 241 -> 268
Other:
- moved on the sheet: C13, C6, C7, C8, D1, D3, D4, D5, R1, R17, R18, R3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

Commit message: Almost routed for 64 pin LPC device
Parts:
- removed F11, F15, F19, F23, F5, F7, F9: 1.25A, 1812, symbol FUSE
- removed FB?: FILTER, symbol FILTER
- removed R4: 10K, symbol R
- removed R40, R41: 560R, symbol R
- removed R42: 120R, symbol R
- removed SW3: DIPS_04, symbol DIPS_04
- removed U2: ADM2484, 16SOIC, symbol ADM2484
- added F2: 1.25A, 1812, symbol FUSE
- added P4, P?: CONN_4, symbol CONN_4
- added P5: CONN_6, symbol CONN_6
- added P?: CONN_5, symbol CONN_5
- added SW4: DIPS_02, symbol DIPS_02
- added U2: ISO3086T, symbol ISO3086T
- C8: value 4u7 -> 10uF
- D2: footprint TO-247 -> DO-214AA; Farnell 1651155 -> 1467550; MFG FAIRCHILD SEMICONDUCTOR - RURG5060 -> (none); PRICE 2 -> .3
- FB1, FB2: renamed from FB?; footprint (none) -> 1806
- R14: value R -> 22k
- R5: value 10K -> 1K
- gave numbers to parts that had none: 1
Connections:
- net labels added: MISO, MOSI, RESET, SCK, SCL, SDA, SSEL, SWCLK, SWDIO
- net labels removed: RESET_SW, V10, V12, V7, V8, V9
- wire segments 268 -> 261
Other:
- note added: "1 = NC\n2 = NC\n3 = A\n4 = VBUS_12V\n5 = VBUS_12V\n6 = B\n7 = BUS_GND\n8 = BUS_GND"
- note removed: "1 = TX+\n2 = TX-\n3 = RX+\n4 = VBUS_12V\n5 = VBUS_12V\n6 = RX-\n7 = BUS_GND\n8 = BUS_GND"
- moved on the sheet: C13, C14, C18, D1, D3, D4, D6, D7, F1, F13, F17, F21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

Commit message: Complete routed version
Parts:
- removed C17: 100nF, symbol C
- removed D8: DIODE, symbol DIODE
- removed P3: POWER, symbol CONN_2
- removed P4: CONN_4, symbol CONN_4
- removed R44, R45: 1k, symbol R
- removed U4: LPC11U35FBD64/401, LQFP64, symbol LPC11U35FBD64/401
- added C23: 100nF, symbol C
- added P3, P8: CONN_4, symbol CONN_4
- added P4: CONN_6, symbol CONN_6
- added R4, R40: 2k2, symbol R
- added U4: LPC11U24FBD48/301, symbol LPC11U24FBD48/301
- C5: value 4u7 -> 10uF
- gave numbers to parts that had none: 2
Connections:
- net labels added: +5VP, BUS_A, BUS_B, BUS_GND, BUS_PWR, DM, DP, USB_DM, USB_DP, VBUS
- net labels removed: UMON
- wire segments 261 -> 217
Other:
- note added: "1 = NC\n2 = NC\n3 = B\n4 = VBUS_12V\n5 = VBUS_12V\n6 = A\n7 = BUS_GND\n8 = BUS_GND"
- note added: "A aka '-' aka TxD-/RxD- aka inverting pin\nB aka '+' aka TxD+/RxD+ aka non-inverting pin"
- note added: "Note: A/B non std. (using TI designation)"
- note removed: "1 = NC\n2 = NC\n3 = A\n4 = VBUS_12V\n5 = VBUS_12V\n6 = B\n7 = BUS_GND\n8 = BUS_GND"
- moved on the sheet: C1, C10, C11, C12, C13, C14, C15, C16, C18, C19, C2, C20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

Commit message: Added extra hole
Parts:
- removed C16: 10000uF, symbol CAPAPOL
Connections:
- wire segments 217 -> 216
Changed lines of the file:
@@
-EESchema Schematic File Version 2  date 5/5/2013 10:57:47 PM
+EESchema Schematic File Version 2  date 5/5/2013 11:23:17 PM
 LIBS:k_lpc1100
 LIBS:kekketek
@@
 	15250 6650 15250 6750
 Wire Wire Line
-	2900 10200 2900 10350
-Wire Wire Line
 	4450 900  3550 900
 Wire Wire Line
@@
 	6550 10200 6550 10250
 Connection ~ 6400 10200
-Connection ~ 2900 10200
 Connection ~ 3300 10750
-Connection ~ 2900 10750
 Wire Wire Line
 	3300 10600 3300 10750
@@
 Text Notes 750  10900 0    60   ~ 0
 Large Cs located close to each USB connector rows
-$Comp
-L CAPAPOL C16
-U 1 1 511BC97B
-P 2900 10550
-F 0 "C16" H 2950 10650 50  0000 L CNN
-F 1 "10000uF" H 2950 10450 50  0000 L CNN
-	1    2900 10550
-	1    0    0    -1
-$EndComp
 Text Label 14750 6750 2    60   ~ 0
 D24

Commit message: Rev 3 PCB layout ok
Parts:
- removed P4: CONN_6, symbol CONN_6
- added P4: CONN_5, symbol CONN_5
- added P9: CONN_4, symbol CONN_4
- added R41: 1k5, symbol R
- C19, C20: value 10000uF -> 4700uF; Farnell (none) -> 1834100
- C2: value 10000uF -> 4700uF; Farnell (none) -> 1834100; PRICE (none) -> 0.4
- FB1, FB2: value 0.1R / 1A -> 0.1R/1A
- R1, R3, R43, R46, R6: value 330R -> 120R
- R10, R9: value 560R -> 1k5
- R11, R12, R20, R21, R22, R23, R24, R25, R26, R27, R28, R29, R30, R31, R32, R33, R34, R35, R36, R37, R38, R39, R7, R8: value 100R -> 120R
- R15: value 1k -> 1k5
- R19: value 10k -> 120R
- R4, R40: value 2k2 -> 1k5
- R5: value 1K -> 1K5
Connections:
- net labels added: ISP_RXD, ISP_TXD, TP1
- net labels removed: COM_nRE
- wire segments 216 -> 221

Commit message: Fixed farnell order codes
Parts:
- C1, C11, C12, C15, C18, C23, C3, C4, C6, C7: footprint (none) -> SM0805; Farnell (none) -> 1759167
- C10, C8, C9: footprint (none) -> SM0805; Farnell (none) -> 1759136
- C13, C14, C21, C22: footprint (none) -> SM0805; Farnell (none) -> 1759194
- C19, C2, C20: footprint (none) -> CP_13x21mm
- C5, R1, R11, R12, R19, R2, R20, R21, R22, R23, R24, R25, R26, R27, R28, R29, R3, R30, R31, R32, R33, R34, R35, R36, R37, R38, R39, R43, R46, R6, R7, R8: footprint (none) -> SM0805
- D1, D3, D4, D6, D7: footprint (none) -> Led_1206
- D2: footprint DO-214AA -> to220-2
- D5: footprint DO-219AB -> SM1812
- F1, F13, F17, F2, F21, F3: footprint 1812 -> SM1812E
- FB1, FB2: footprint 1806 -> SM1812
- J13, J14: footprint (none) -> RJ45_8; Farnell (none) -> 2135979
- J15: footprint (none) -> conn_usb_B_micro_smd; Farnell (none) -> 1568026
- JP1: footprint (none) -> pin_strip_2
- P1, P2: footprint (none) -> mstba_2,5/2-g-5,08
- P3, P7, P8, P9: footprint (none) -> pin_strip_4
- P4, P6: footprint (none) -> pin_strip_5
- P5: footprint (none) -> pin_strip_6
- Q1: footprint SOT-23 -> SOT23
- R10, R15, R16, R4, R40, R41, R5, R9: footprint (none) -> SM0805; Farnell (none) -> 2074373
- R13, R14: footprint (none) -> SM0805; Farnell (none) -> 9332820
- R17, R18: footprint (none) -> SM0805; Farnell (none) -> 9233822
- SW1, SW2: footprint (none) -> PCB_PUSH; Farnell (none) -> 1656423
- SW4: footprint (none) -> dip_2-300; Farnell (none) -> 1523994
- U1, U3: footprint SOT-223 -> SOT223
- U2: footprint (none) -> soic-16; Farnell (none) -> 2057088
- U4: footprint (none) -> lqfp48
- VR1: footprint 1206 -> SM1206POL
- X1: footprint (none) -> crystal_hc-49/smd; Farnell (none) -> 9713344
